Commit message: modify simulation

File: Gazebo/usv_gazebo/urdf/camera_gazebo.xacro (robot description, xacro)
@@ -5,10 +5,10 @@
   <gazebo reference="camera_link">
     <sensor type="camera" name="camera1">
-      <update_rate>30.0</update_rate>
+      <update_rate>1.0</update_rate>
       <camera name="head">
         <horizontal_fov>1.04712042</horizontal_fov>
         <image>
-          <width>1296</width>
-          <height>964</height>
+          <width>640</width>
+          <height>480</height>
           <format>R8G8B8</format>
         </image>

File: Gazebo/usv_gazebo/urdf/gps_gazebo.xacro (robot description, xacro)
@@ -4,9 +4,9 @@
     <gazebo>
       <plugin name="gps_plugin_${name}" filename="libhector_gazebo_ros_gps.so">
-          <updateRate>1.0</updateRate>
+          <updateRate>20.0</updateRate>
 		      <alwaysOn>true</alwaysOn>
           <bodyName>base_link</bodyName>
           <frameId>base_link</frameId>
-          <topicName>/gps/fix</topicName>
+          <topicName>/gps</topicName>
           <velocityTopicName>/gps/fix_velocity</velocityTopicName>
           <referenceLatitude>-30.06022459407145675</referenceLatitude>

File: Gazebo/usv_gazebo/urdf/laser_gazebo.xacro (robot description, xacro)
@@ -7,5 +7,5 @@
       <pose>0 0 0 0 0 0</pose>
       <visualize>false</visualize>
-      <update_rate>40</update_rate>
+      <update_rate>5</update_rate>
       <ray>
         <scan>

File: Gazebo/usv_gazebo/urdf/usv_gazebo_laser.xacro (robot description, xacro)
@@ -31,9 +31,9 @@
   <!-- <xacro:if value="$(arg p3d)">
     <xacro:usv_p3d_gazebo name="usv"/>
-  </xacro:if> -->
+  </xacro:if>  samples="1875"-->
   <xacro:usv_gazebo_camera name="usv"/>
-  <xacro:include filename="$(find velodyne_description)/urdf/HDL-32E.urdf.xacro"/>
-  <HDL-32E parent="base_link" name="velodyne" topic="/velodyne_points2" hz="10" samples="220">
-        <origin xyz="0 0 0.6" rpy="0 0 0" />
-  </HDL-32E>
+  <xacro:include filename="$(find velodyne_description)/urdf/VLP-16.urdf.xacro"/>
+  <VLP-16 parent="base_link" name="velodyne" topic="/velodyne_points2" hz="1">
+        <origin xyz="0 0 0.5" rpy="0 0 0" />
+  </VLP-16>
 </robot>

File: Gazebo/usv_gazebo/urdf/usv_urdf.xacro (robot description, xacro)
@@ -83,5 +83,5 @@
   <joint name="camera_joint" type="fixed">
     <axis xyz="0 1 0" />
-    <origin xyz="0.32 0 0.5" rpy="0 0 0"/>
+    <origin xyz="0.0 0 0.4" rpy="0 0 0"/>
     <parent link="base_link"/>
     <child link="camera_link"/>

Commit message: add exp env

File: Gazebo/usv_gazebo/urdf/camera_gazebo.xacro (robot description, xacro)
@@ -3,5 +3,5 @@
   <xacro:macro name="usv_gazebo_camera" params="name">
   <!-- camera -->
-  <gazebo reference="camera_link">
+  <gazebo reference="${name}/camera_link">
     <sensor type="camera" name="camera1">
       <update_rate>1.0</update_rate>
@@ -30,7 +30,7 @@
         <updateRate>0.0</updateRate>
         <cameraName>camera</cameraName>
-        <imageTopicName>image_raw</imageTopicName>
-        <cameraInfoTopicName>camera_info</cameraInfoTopicName>
-        <frameName>camera_link</frameName>
+        <imageTopicName>${name}/image_raw</imageTopicName>
+        <cameraInfoTopicName>${name}/camera_info</cameraInfoTopicName>
+        <frameName>${name}/camera_link</frameName>
         <hackBaseline>0.07</hackBaseline>
         <distortionK1>0.0</distortionK1>

File: Gazebo/usv_gazebo/urdf/gps_gazebo.xacro (robot description, xacro)
@@ -6,10 +6,10 @@
           <updateRate>20.0</updateRate>
 		      <alwaysOn>true</alwaysOn>
-          <bodyName>base_link</bodyName>
-          <frameId>base_link</frameId>
-          <topicName>/gps</topicName>
-          <velocityTopicName>/gps/fix_velocity</velocityTopicName>
-          <referenceLatitude>-30.06022459407145675</referenceLatitude>
-          <referenceLongitude>-51.173913575780311191</referenceLongitude>
+          <bodyName>${name}/base_link</bodyName>
+          <frameId>${name}/base_link</frameId>
+          <topicName>${name}/gps</topicName>
+          <velocityTopicName>${name}/gps/fix_velocity</velocityTopicName>
+          <referenceLatitude>30.06022459407145675</referenceLatitude>
+          <referenceLongitude>120.173913575780311191</referenceLongitude>
           <referenceHeading>90</referenceHeading>
           <referenceAltitude>10</referenceAltitude>

File: Gazebo/usv_gazebo/urdf/imu_gazebo.xacro (robot description, xacro)
@@ -7,8 +7,8 @@
     <plugin name="imu_plugin_${name}" filename="libgazebo_ros_imu.so">
       <alwaysOn>true</alwaysOn>
-      <bodyName>base_link</bodyName>
-      <frameName>base_link</frameName>
-      <topicName>imu</topicName>
-      <serviceName>imu_service</serviceName>
+      <bodyName>${name}/base_link</bodyName>
+      <frameName>${name}/base_link</frameName>
+      <topicName>${name}/imu</topicName>
+      <serviceName>${name}/imu_service</serviceName>
       <gaussianNoise>0.0</gaussianNoise>
       <updateRate>20.0</updateRate>

File: Gazebo/usv_gazebo/urdf/usv_gazebo_base.xacro (robot description, xacro)
@@ -2,34 +2,27 @@
 <robot xmlns:xacro="http://ros.org/wiki/xacro"
        name="usv">
+  <xacro:property name="namespace" value="$(arg name)"/>
   <!-- Defines the "usv_base" macro -->
-  <xacro:include filename="$(find usv_gazebo)/urdf/usv_urdf.xacro" />
+  <xacro:include filename="$(find usv_gazebo)/urdf/usv_urdf2.xacro" />
   <!--<xacro:include filename="$(find usv_gazebo)/urdf/usv_urdf_camera.xacro" />-->
   <!-- Defines the "usv_gazebo" macro which implements the plugin for USV dynamics -->
-  <xacro:include filename="$(find usv_gazebo_plugins)/urdf/usv_gazebo_dynamics_plugin.xacro" />
+  <xacro:include filename="$(find usv_gazebo_plugins)/urdf/usv_gazebo_dynamics_plugin2.xacro" />
   <!-- Testing old plugin -->
   <!--<xacro:include filename="$(find usv_plugins)/urdf/usv_plugin.xacro" />-->
-  <!-- Defines the macro for including simulated camera -->
-  <xacro:include filename="$(find usv_gazebo)/urdf/camera_gazebo.xacro" />
   <!-- Defines the macro for simulated GPS -->
   <xacro:include filename="$(find usv_gazebo)/urdf/gps_gazebo.xacro" />
   <!-- Defines the macro for simulated IMU -->
   <xacro:include filename="$(find usv_gazebo)/urdf/imu_gazebo.xacro" />
-  <!-- Macro for P3D ground truth -->
-  <!-- <xacro:include filename="$(find usv_gazebo)/urdf/p3d_gazebo.xacro" /> -->
   <!-- Call the macros defined above -->
   <!-- includes basic description witout plugins -->
-  <xacro:usv_base />
+  <xacro:usv_base name="${namespace}"/>
   <!-- USV dynamic model -->
-  <xacro:usv_gazebo name="usv"/>
+  <xacro:usv_gazebo name="${namespace}"/>
   <!-- Optional sensor plugins - called by macros defined above -->
   <xacro:if value="$(arg gps)">
-    <xacro:usv_gps_gazebo name="usv"/>
+    <xacro:usv_gps_gazebo  name="${namespace}"/>
   </xacro:if>
   <xacro:if value="$(arg imu)">
-    <xacro:usv_imu_gazebo name="usv"/>
+    <xacro:usv_imu_gazebo  name="${namespace}"/>
   </xacro:if>
-  <!-- <xacro:if value="$(arg p3d)">
-    <xacro:usv_p3d_gazebo name="usv"/>
-  </xacro:if> -->
-  <xacro:usv_gazebo_camera name="usv"/>
 </robot>

File: Gazebo/usv_gazebo/urdf/usv_gazebo_laser.xacro (robot description, xacro)
@@ -2,4 +2,5 @@
 <robot xmlns:xacro="http://ros.org/wiki/xacro"
        name="usv">
+  <xacro:property name="namespace" value="$(arg name)"/>
   <!-- Defines the "usv_base" macro -->
   <xacro:include filename="$(find usv_gazebo)/urdf/usv_urdf.xacro" />
@@ -16,24 +17,24 @@
   <xacro:include filename="$(find usv_gazebo)/urdf/imu_gazebo.xacro" />
   <!-- Macro for P3D ground truth -->
-  <!-- <xacro:include filename="$(find usv_gazebo)/urdf/p3d_gazebo.xacro" /> -->
+  <xacro:include filename="$(find velodyne_description)/urdf/VLP-16.urdf.xacro"/>
   <!-- Call the macros defined above -->
   <!-- includes basic description witout plugins -->
-  <xacro:usv_base />
+  <xacro:usv_base  name="${namespace}"/>
   <!-- USV dynamic model -->
-  <xacro:usv_gazebo name="usv"/>
+  <xacro:usv_gazebo  name="${namespace}"/>
   <!-- Optional sensor plugins - called by macros defined above -->
   <xacro:if value="$(arg gps)">
-    <xacro:usv_gps_gazebo name="usv"/>
+    <xacro:usv_gps_gazebo  name="${namespace}"/>
   </xacro:if>
   <xacro:if value="$(arg imu)">
-    <xacro:usv_imu_gazebo name="usv"/>
+    <xacro:usv_imu_gazebo  name="${namespace}"/>
   </xacro:if>
-  <!-- <xacro:if value="$(arg p3d)">
-    <xacro:usv_p3d_gazebo name="usv"/>
-  </xacro:if>  samples="1875"-->
-  <xacro:usv_gazebo_camera name="usv"/>
-  <xacro:include filename="$(find velodyne_description)/urdf/VLP-16.urdf.xacro"/>
-  <VLP-16 parent="base_link" name="velodyne" topic="/velodyne_points2" hz="1">
+  <xacro:if value="$(arg camera)">
+    <xacro:usv_gazebo_camera  name="${namespace}"/>
+  </xacro:if>
+  <xacro:if value="$(arg p3d)">
+  <VLP-16 parent="${namespace}/base_link" name="velodyne" topic="/velodyne_points2" hz="2">
         <origin xyz="0 0 0.5" rpy="0 0 0" />
   </VLP-16>
+  </xacro:if>
 </robot>

File: Gazebo/usv_gazebo/urdf/usv_urdf2.xacro (robot description, xacro)
@@ -80,8 +80,9 @@
   </gazebo>
   <!-- Define a location for the camera to sit -->
-  <xacro:property name="camera_size" value="0.05" /> <!-- Size of square 'camera' box -->
+  <xacro:property name="camera_size_h" value="1" /> <!-- Size of square 'camera' box -->
+  <xacro:property name="camera_size_w" value="1" />
   <joint name="${name}/camera_joint" type="fixed">
     <axis xyz="0 1 0" />
-    <origin xyz="0.0 0 0.4" rpy="0 0 0"/>
+    <origin xyz="0.0 0 0.5" rpy="0 0 0"/>
     <parent link="${name}/base_link"/>
     <child link="${name}/camera_link"/>
@@ -91,5 +92,5 @@
       <origin xyz="0 0 0" rpy="0 0 0"/>
       <geometry>
-	      <box size="${camera_size} ${camera_size} ${camera_size}"/>
+	      <box size="${camera_size_w} ${camera_size_w} ${camera_size_h}"/>
       </geometry>
     </collision>
@@ -97,7 +98,7 @@
       <origin xyz="0 0 0" rpy="0 0 0"/>
       <geometry>
-	      <box size="${camera_size} ${camera_size} ${camera_size}"/>
+	      <box size="${camera_size_w} ${camera_size_w} ${camera_size_h}"/>
       </geometry>
-      <material name="red"/>
+      <material name="black"/>
     </visual>
     <inertial>

File: Gazebo/usv_gazebo_plugins/urdf/usv_gazebo_dynamics_plugin2.xacro (robot description, xacro)
@@ -32,5 +32,5 @@
 		<metacentricLength>0.4</metacentricLength>
 		<metacentricWidth>0.4</metacentricWidth>
-      </plugin>
+	  </plugin>
     </gazebo>
   </xacro:macro>
